File: pogger power.kicad_pcb (KiCad board)
At the start: 2 copper layers, 49.5 x 51.4 mm, 34 parts, among them J1 Conn_01x01_Female, J2 Conn_01x01_Female, J3 Conn_01x01_Female, J4 Conn_01x01_Female, J5 Conn_01x01_Female, J6 Conn_01x01_Female, Q1 FDBL86361-F085, Q2 BSS84, U1 L78L05_SO8, U2 LT3757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

Commit message: added silkscreen labels
Other:
- board text added: "+60V"
- board text added: "GND"
- board text added: "VIN"
- board text added: "dcdc.poggies.net"
Changed lines of the file:
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@@
   (general
     (thickness 1.6)
-    (drawings 5)
+    (drawings 12)
     (tracks 277)
     (zones 0)
@@
   (layers
     (0 F.Cu signal)
-    (31 B.Cu signal hide)
+    (31 B.Cu signal)
     (32 B.Adhes user)
     (33 F.Adhes user)
     (34 B.Paste user)
     (35 F.Paste user)
-    (36 B.SilkS user hide)
+    (36 B.SilkS user)
     (37 F.SilkS user)
     (38 B.Mask user)
@@
     )
   )
-  (gr_text nb2020 (at 156.21 85.344) (layer F.SilkS)
+  (gr_text dcdc.poggies.net (at 146.7485 92.456) (layer B.SilkS)
+    (effects (font (size 1 1) (thickness 0.15)) (justify mirror))
+  )
+  (gr_text GND (at 165.1 96.266) (layer B.SilkS)
+    (effects (font (size 3 3) (thickness 0.3)) (justify mirror))
+  )
+  (gr_text GND (at 128.524 96.266) (layer B.SilkS)
+    (effects (font (size 3 3) (thickness 0.3)) (justify mirror))
+  )
+  (gr_text +60V (at 157.893 120.65) (layer B.SilkS)
+    (effects (font (size 3 3) (thickness 0.3)) (justify mirror))
+  )
+  (gr_text GND (at 133.938 120.904) (layer B.SilkS)
+    (effects (font (size 3 3) (thickness 0.3)) (justify mirror))
+  )
+  (gr_text GND (at 133.938 77.724) (layer B.SilkS)
+    (effects (font (size 3 3) (thickness 0.3)) (justify mirror))
+  )
+  (gr_text VIN (at 157.893 77.978) (layer B.SilkS)
+    (effects (font (size 3 3) (thickness 0.3)) (justify mirror))
+  )
+  (gr_text nb2020 (at 159.512 85.344) (layer F.SilkS)
     (effects (font (size 1 1) (thickness 0.15)))
   )

Commit message: fixed footprint of output ceramic caps
Parts:
- C5, C9: footprint Capacitor_SMD:C_1206_3216Metric_Pad1.42x1.75mm_HandSolder -> Capacitor_SMD:C_1210_3225Metric_Pad1.42x2.65mm_HandSolder
